File: HW/Underglow-slave/Underglow-slave.kicad_pcb (KiCad board)
At the start: 2 copper layers, 3 parts, among them U1 CH572Q

Commit message: claude did something
Parts:
- removed ADDR_LED1: ~, Mylib:Addressable_led_adapter_10mm
- added C1: 10uF 25V, Capacitor_SMD:C_0805_2012Metric, F.Cu at (122.6, 114.0)
- added C10: 100nF, Capacitor_SMD:C_0402_1005Metric, F.Cu at (127.5, 114.6)
- added C11: 100nF, Capacitor_SMD:C_0402_1005Metric, F.Cu at (138.0, 114.6)
- added C12: 100nF, Capacitor_SMD:C_0402_1005Metric, F.Cu at (148.5, 114.6)
- added C2: 10uF 10V, Capacitor_SMD:C_0603_1608Metric, F.Cu at (115.5, 117.2)
- added C3: 1uF, Capacitor_SMD:C_0402_1005Metric, F.Cu at (111.0, 116.8)
- added C4: 2.2uF, Capacitor_SMD:C_0402_1005Metric, F.Cu at (106.4, 114.4)
- added C5: 100nF, Capacitor_SMD:C_0402_1005Metric, F.Cu at (107.4, 114.4)
- added C8: DNP, Capacitor_SMD:C_0402_1005Metric, F.Cu at (106.9, 108.9)
- added C9: DNP, Capacitor_SMD:C_0402_1005Metric, F.Cu at (103.5, 108.9)
- added D1: B5819W, Diode_SMD:D_SOD-123, F.Cu at (154.8, 110.0)
- added D2: WS2815B-V1, LED_SMD:LED_WS2812_PLCC6_5.0x5.0mm_P1.6mm, F.Cu at (127.5, 110.0)
- added D3: WS2815B-V1, LED_SMD:LED_WS2812_PLCC6_5.0x5.0mm_P1.6mm, F.Cu at (138.0, 110.0)
- added D4: WS2815B-V1, LED_SMD:LED_WS2812_PLCC6_5.0x5.0mm_P1.6mm, F.Cu at (148.5, 110.0)
- added D5: WS2815B-V1, LED_SMD:LED_WS2812_PLCC6_5.0x5.0mm_P1.6mm, B.Cu at (148.5, 110.0)
- added D6: WS2815B-V1, LED_SMD:LED_WS2812_PLCC6_5.0x5.0mm_P1.6mm, B.Cu at (138.0, 110.0)
- added D7: WS2815B-V1, LED_SMD:LED_WS2812_PLCC6_5.0x5.0mm_P1.6mm, B.Cu at (127.5, 110.0)
- added H1: MountingHole, MountingHole:MountingHole_2.2mm_M2, F.Cu at (154.8, 103.3)
- added H2: MountingHole, MountingHole:MountingHole_2.2mm_M2, F.Cu at (154.8, 116.7)
- added J1: PROG, TreeGlow:ProgPads_1x05_P2.54mm, B.Cu at (109.6, 118.0)
- added J2: PWR 12V, Connector_Wire:SolderWire-0.75sqmm_1x04_P4.8mm_D1.25mm_OD2.3mm, F.Cu at (159.3, 102.8)
- added J3: LED DO, TestPoint:TestPoint_Pad_D1.5mm, B.Cu at (122.2, 108.4)
- added R1: 1.5k, Capacitor_SMD:C_0402_1005Metric, F.Cu at (107.6, 116.2)
- added R2: 0R, Capacitor_SMD:C_0402_1005Metric, F.Cu at (105.2, 108.0)
- added R3: 33R, Capacitor_SMD:C_0402_1005Metric, F.Cu at (113.0, 113.7)
- added U2: HT7550-1, Package_TO_SOT_SMD:SOT-89-3, F.Cu at (119.2, 113.4)
- added Y1: 32MHz, Crystal:Crystal_SMD_3225-4Pin_3.2x2.5mm, F.Cu at (113.6, 108.6)
- AE1: value Antenna -> PCB IFA
- U1: footprint Package_DFN_QFN:DFN-10-1EP_2.6x2.6mm_P0.5mm_EP1.3x2.2mm -> Package_DFN_QFN:DFN-10-1EP_3x3mm_P0.5mm_EP1.7x2.5mm
- moved U1 99.1 mm to (109.5, 111.5), turned to 90 degrees
- moved AE1 94.3 mm to (103.5, 106.0)
Connections:
- AE1 pad 1: Net-(AE1-A) -> /RF_ANT
- AE1 pad 2: (no net) -> GND
- U1 pad 1: +3.3V -> /VDD33
- U1 pad 10: Net-(AE1-A) -> /RF_CHIP
- U1 pad 11: (no net) -> GND
- U1 pad 5: /LED_RGB -> /LED_DATA_MCU
- U1 pad 6: /RX -> /UART_TX
- U1 pad 7: /TX -> unconnected-(U1-PA3/TXD/PWM3-Pad7)
- U1 pad 8: /XOUT -> /XO
- U1 pad 9: /XIN -> /XI
Routing:
- net GND: track 0.00 -> 226.9 mm, vias 0 -> 26
- net +12V: track 0.00 -> 75.2 mm, vias 0 -> 3
- net +5V: track 0.00 -> 22.9 mm, vias 0 -> 1
- net /VIN_12V: track 0.00 -> 22.6 mm
- net /LED_D1: track 0.00 -> 16.9 mm
- net /UART_TX: track 0.00 -> 9.80 mm, vias 0 -> 1
- net /SWDIO: track 0.00 -> 8.04 mm, vias 0 -> 1
- net /XO: track 0.00 -> 7.49 mm
- net /SWCLK: track 0.00 -> 7.44 mm, vias 0 -> 1
- net /VDD33: track 0.00 -> 6.31 mm
- net /XI: track 0.00 -> 6.29 mm
- net /LED_D6: track 0.00 -> 5.60 mm
- net /LED_D2: track 0.00 -> 5.60 mm
- net /LED_D5: track 0.00 -> 5.60 mm
- net /LED_D3: track 0.00 -> 5.60 mm
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- added copper zone on B.Cu, net GND
- added copper zone on F.Cu, net GND
Other:
- board outline added: 62 x 20 mm
- board text added: "+12V"
- board text added: "DO"
- board text added: "GND"
- board text added: "TreeGlow node (back)"
- board text added: "TreeGlow node v1.0"
