File: HW/Underglow-slave/Underglow-slave.kicad_pcb (KiCad board)
At the start: 2 copper layers, 3 parts, among them U1 CH572Q

Commit message: stuff works
claude rewrote it
Parts:
- added C1: DNP, Capacitor_SMD:C_0402_1005Metric, F.Cu at (108.6, 112.6)
- added C2: DNP, Capacitor_SMD:C_0402_1005Metric, F.Cu at (110.6, 112.6)
- added C3: DNP, Capacitor_SMD:C_0402_1005Metric, F.Cu at (107.6, 107.6)
- added C4: 1u 25V, Capacitor_SMD:C_0603_1608Metric, F.Cu at (113.0, 111.8)
- added C5: 1u, Capacitor_SMD:C_0402_1005Metric, F.Cu at (102.4, 111.8)
- added C6: 2.2u, Capacitor_SMD:C_0402_1005Metric, F.Cu at (102.4, 109.4)
- added C7: 100n, Capacitor_SMD:C_0402_1005Metric, F.Cu at (102.4, 110.6)
- added H1: GND screw, MountingHole:MountingHole_3.2mm_M3_Pad_Via, F.Cu at (118.3, 110.9)
- added J1: Debug_header, Connector_PinHeader_1.27mm:PinHeader_1x04_P1.27mm_Vertical, F.Cu at (106.2, 117.6)
- added TP1: +12V in, TestPoint:TestPoint_THTPad_3.0x3.0mm_Drill1.5mm, F.Cu at (119.6, 117.2)
- added U2: HT7550-1, Package_TO_SOT_SMD:SOT-89-3, F.Cu at (114.6, 116.8)
- added Y1: 32MHz 8pF, Crystal:Crystal_SMD_2016-4Pin_2.0x1.6mm, F.Cu at (109.4, 110.4)
- moved ADDR_LED1 100.3 mm to (100.8, 130.3)
- moved U1 96.0 mm to (105.5, 110.5)
- moved AE1 95.2 mm to (105.0, 106.0)
Connections:
- AE1 pad 2: (no net) -> GND
- U1 pad 11: (no net) -> GND
Routing:
- added copper zone on B.Cu, net GND
- added copper zone on F.Cu, net GND
Other:
- board outline added: 22 x 31 mm
