File: HW/Underglow-slave/Underglow-slave.kicad_sch (KiCad schematic)
At the start: 8 parts, among them J1 Debug_header, U1 CH572Q, Y1 Crystal

Commit message: stuff works
claude rewrote it
Parts:
- added C4: 1u 25V, Capacitor_SMD:C_0603_1608Metric, symbol Device:C_Small
- added C5: 1u, Capacitor_SMD:C_0402_1005Metric, symbol Device:C_Small
- added C6: 2.2u, Capacitor_SMD:C_0402_1005Metric, symbol Device:C_Small
- added C7: 100n, Capacitor_SMD:C_0402_1005Metric, symbol Device:C_Small
- added H1: GND screw, MountingHole:MountingHole_3.2mm_M3_Pad_Via, symbol Mechanical:MountingHole_Pad
- added J2: PWM_out, Connector_PinHeader_1.27mm:PinHeader_1x04_P1.27mm_Vertical, symbol Connector_Generic:Conn_01x04
- added TP1: +12V in, TestPoint:TestPoint_THTPad_3.0x3.0mm_Drill1.5mm, symbol Connector:TestPoint
- added U2: HT7550-1, Package_TO_SOT_SMD:SOT-89-3, symbol Regulator_Linear:HT75xx-1-SOT89
- AE1: symbol Device:Antenna -> Device:Antenna_Shield
- C1, C2, C3: value C_Small -> DNP; footprint (none) -> Capacitor_SMD:C_0402_1005Metric; now not fitted
- J1: footprint (none) -> Connector_PinHeader_1.27mm:PinHeader_1x04_P1.27mm_Vertical
- Y1: value Crystal -> 32MHz 8pF; footprint (none) -> Crystal:Crystal_SMD_2016-4Pin_2.0x1.6mm; symbol Device:Crystal -> Device:Crystal_GND24
Connections:
- net +12V: now also C4.1, TP1.1, U2.2 (VIN)
- net +3.3V: now also C6.1, C7.1
- net +5V: now also C5.1, U2.3 (VOUT)
- net GND: now also AE1.2 (Shield), U1.11 (GND), Y1.2 (G), Y1.4 (G), C4.2, C5.2, C6.2, C7.2, H1.1, J2.4 (Pin_4), U2.1 (GND); no longer U1.0 (GND)
- net LED_RGB: now also J2.1 (Pin_1)
- net XOUT: now also Y1.3; no longer Y1.2
- net RX renamed PWM2
- net PWM2: now also J2.2 (Pin_2)
- net TX renamed PWM3
- net PWM3: now also J2.3 (Pin_3)
